File: USB/USB.kicad_pcb (KiCad board)
At the start: 2 copper layers, 54.6 x 31 mm, 41 parts, among them J1 Conn_02x12_Odd_Even, J2 CONN, Q1 2N7002, U1 TSOP17xx

Commit message: added background silkscreen J2 connector pins
Other:
- board text added: "+3V3"
Changed lines of the file:
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@@
   (general
     (thickness 1.6)
-    (drawings 64)
+    (drawings 69)
     (tracks 444)
     (zones 0)
@@
   (page A4)
   (layers
-    (0 F.Cu signal)
+    (0 F.Cu signal hide)
     (31 B.Cu signal)
     (32 B.Adhes user)
-    (33 F.Adhes user)
+    (33 F.Adhes user hide)
     (34 B.Paste user)
-    (35 F.Paste user)
+    (35 F.Paste user hide)
     (36 B.SilkS user)
-    (37 F.SilkS user)
+    (37 F.SilkS user hide)
     (38 B.Mask user)
-    (39 F.Mask user)
-    (40 Dwgs.User user)
-    (41 Cmts.User user)
-    (42 Eco1.User user)
+    (39 F.Mask user hide)
+    (40 Dwgs.User user hide)
+    (41 Cmts.User user hide)
+    (42 Eco1.User user hide)
     (43 Eco2.User user)
     (44 Edge.Cuts user)
@@
     (46 B.CrtYd user)
     (47 F.CrtYd user)
-    (48 B.Fab user)
-    (49 F.Fab user)
+    (48 B.Fab user hide)
+    (49 F.Fab user hide)
   )
   (setup
@@
       (xy -0.035487 4.576309) (xy -0.011682 4.575626)) (layer B.SilkS) (width 0.01))
   )
+  (gr_text GND (at 170.434 106.83) (layer B.SilkS)
+    (effects (font (size 0.5 0.5) (thickness 0.125)) (justify mirror))
+  )
+  (gr_text GP27 (at 170.434 104.29) (layer B.SilkS)
+    (effects (font (size 0.5 0.5) (thickness 0.125)) (justify mirror))
+  )
+  (gr_text GN27 (at 170.434 101.75) (layer B.SilkS)
+    (effects (font (size 0.5 0.5) (thickness 0.125)) (justify mirror))
+  )
+  (gr_text +3V3 (at 170.434 99.21) (layer B.SilkS)
+    (effects (font (size 0.5 0.5) (thickness 0.125)) (justify mirror))
+  )
+  (gr_text +5V (at 170.434 96.67) (layer B.SilkS)
+    (effects (font (size 0.5 0.5) (thickness 0.125)) (justify mirror))
+  )
   (target plus (at 119.634 109.728) (size 5) (width 0.05) (layer Edge.Cuts))
